File: KiCad Files/OEM_PHOB1.X/bpad_PCB_phob1X_OEM.kicad_pcb (KiCad board)
At the start: 2 copper layers, 31.6 x 51.6 mm, 28 parts, among them J1 Conn_01x04, SW1 C_left, SW2 C_up, SW3 C_down, SW4 C_right

Commit message: Fix
Routing:
- net /C_x: track 78.7 -> 80.5 mm
Changed lines of the file:
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@@
   (segment (start 124 101.3) (end 122.6 99.9) (width 0.4) (layer "B.Cu") (net 2))
   (segment (start 133.87 120.54) (end 134.12 120.79) (width 0.6) (layer "F.Cu") (net 3))
+  (segment (start 129.423 98.669) (end 124.831 98.669) (width 0.6) (layer "F.Cu") (net 3))
   (segment (start 133.87 117.54) (end 133.87 114.54) (width 0.6) (layer "F.Cu") (net 3))
   (segment (start 133.87 114.54) (end 134.12 114.29) (width 0.6) (layer "F.Cu") (net 3))
-  (segment (start 138.87 102.88) (end 135.29 99.3) (width 0.6) (layer "F.Cu") (net 3))
   (segment (start 123.3125 97.3125) (end 123.3125 98.1) (width 0.4) (layer "F.Cu") (net 3))
-  (segment (start 135.29 99.3) (end 124.2 99.3) (width 0.6) (layer "F.Cu") (net 3))
   (segment (start 138.87 102.88) (end 138.62 102.63) (width 0.6) (layer "F.Cu") (net 3))
   (segment (start 123.4125 98.1) (end 123.3125 98.2) (width 0.6) (layer "F.Cu") (net 3))
   (segment (start 133.87 117.54) (end 133.87 120.54) (width 0.6) (layer "F.Cu") (net 3))
+  (segment (start 130.175 97.917) (end 129.423 98.669) (width 0.6) (layer "F.Cu") (net 3))
   (segment (start 138.62 102.63) (end 138.62 99.63) (width 0.6) (layer "F.Cu") (net 3))
+  (segment (start 138.87 102.88) (end 138.87 101.913) (width 0.6) (layer "F.Cu") (net 3))
+  (segment (start 138.87 101.913) (end 134.874 97.917) (width 0.6) (layer "F.Cu") (net 3))
+  (segment (start 123.8 99.7) (end 123.4125 99.7) (width 0.6) (layer "F.Cu") (net 3))
   (segment (start 121.53 82.27) (end 121.53 95.53) (width 0.4) (layer "F.Cu") (net 3))
   (segment (start 121.53 95.53) (end 123.3125 97.3125) (width 0.4) (layer "F.Cu") (net 3))
+  (segment (start 134.874 97.917) (end 130.175 97.917) (width 0.6) (layer "F.Cu") (net 3))
   (segment (start 125.8 78) (end 121.53 82.27) (width 0.4) (layer "F.Cu") (net 3))
+  (segment (start 124.831 98.669) (end 123.8 99.7) (width 0.6) (layer "F.Cu") (net 3))
   (segment (start 138.87 102.88) (end 138.87 105.88) (width 0.6) (layer "F.Cu") (net 3))
-  (segment (start 124.2 99.3) (end 123.8 99.7) (width 0.6) (layer "F.Cu") (net 3))
   (segment (start 131.28 100.5) (end 131.28 99.3) (width 0.6) (layer "F.Cu") (net 3))
-  (segment (start 123.8 99.7) (end 123.4125 99.7) (width 0.6) (layer "F.Cu") (net 3))
   (segment (start 123.3125 98.2) (end 123.3125 99.7) (width 0.6) (layer "F.Cu") (net 3))
   (segment (start 127.1888 77.9924) (end 128.016 77.9924) (width 0.25) (layer "F.Cu") (net 3))

Commit message: cleaned up and fixed
Routing:
- net /C_x: track 80.5 -> 83.1 mm
- net /C_y: track 73.9 -> 73.6 mm, vias 2 -> 3
